Commit message: all files uploaded

File: cart_description/cart other files/robot.urdf (robot description, URDF)
Before this commit: robot cart, 7 links, 6 joints
Links:
- removed link laser_frame
- link base_link: geometry collision box size=1 .5 .15; visual box size=1 .5 .15
Joints:
- removed joint laser_joint

File: cart_description/urdf/cart.urdf.xacro (robot description, xacro)
@@ -3,4 +3,4 @@
     <xacro:include filename="cart_design.xacro" />
     <xacro:include filename="cart_control.gazebo"/>
-    <xacro:include filename="lidar.xacro" />
+    <!-- <xacro:include filename="lidar.xacro" /> -->
 </robot>

File: cart_navigation/urdf/cart_design.xacro (robot description, xacro)
@@ -1,16 +1,10 @@
 <?xml version='1.0'?>
 <robot name="cart" xmlns:xacro="http://www.ros.org/wiki/xacro">
-  <xacro:include filename="$(find cart_navigation)/urdf/inertial_macros.xacro" />
-  <!-- STEP 5 - Gazebo plugin -->
   <xacro:include filename="$(find cart_navigation)/urdf/cart_control.gazebo" />
-   <!-- STEP 4 - RViz colors -->
   <xacro:include filename="$(find cart_navigation)/urdf/material.xacro" />
-  <!-- STEP 1 - Robot footprint -->
-  <link name="base_footprint">
-  </link>
-  <!-- STEP 2 - Robot chassis = base_link -->
+  <link name="base_footprint" />
   <joint name="base_footprint_joint" type="fixed">
-    <origin xyz="0 0 -0.075" rpy="0 0 0" />
-    <parent link="base_footprint"/>
+    <origin xyz="0 0 0" rpy="0 0 0" />
+    <parent link="base_footprint" />
     <child link="base_link" />
   </joint>
@@ -18,232 +12,231 @@
     <pose>0 0 0 0 0 0</pose>
     <inertial>
-      <mass value="15.0"/>
-      <origin xyz="0.0 0 0" rpy=" 0 0 0"/>
-      <inertia
-          ixx="0.0625" ixy="0" ixz="0"
-          iyy="0.2125" iyz="0"
-          izz="0.25"
-      />
+      <mass value="9.0" />
+      <origin xyz="0.0 0 0" rpy="0 0 0" />
+      <inertia ixx="0.204375" ixy="0" ixz="0" iyy="0.766875" iyz="0" izz="0.9375" />
     </inertial>
     <collision name='collision'>
-      <origin xyz="0 0 0" rpy=" 0 0 0"/>
-      <geometry>
-        <box size="1 .5 .15"/>
+      <origin xyz="0 0 0" rpy="0 0 0" />
+      <geometry>
+        <box size="1 .5 .15" />
       </geometry>
     </collision>
     <visual name='base_link_visual'>
-      <origin xyz="0 0 0" rpy=" 0 0 0"/>
-      <geometry>
-        <box size="1 .5 .15"/>
+      <origin xyz="0 0 0" rpy="0 0 0" />
+      <geometry>
+        <box size="1 .5 .15" />
       </geometry>
       <material name="grey">
-        <color rgba="0.5 0.5 0.5 1.0"/>
-      </material>
-    </visual>
-  </link>
-  <!-- Stand Panel -->
-  <!-- <link name="stand_panel">
-    <inertial>
-      <mass value="1"/>
-      <inertia ixx="0.166667" iyy="0.166667" izz="0.166667" ixy="0" ixz="0" iyz="0"/>
+        <color rgba="0.5 0.5 0.5 1.0" />
+      </material>
+    </visual>
+  </link>
+  <joint type="continuous" name="front_left_wheel_joint">
+    <origin xyz="0.35 0.3 0" rpy="0 0 0" />
+    <child link="front_left_wheel" />
+    <parent link="base_link" />
+    <axis xyz="0 1 0" rpy="0 0 0" />
+    <limit effort="100" velocity="10" />
+    <dynamics damping="3.0" friction="3.0" />
+  </joint>
+  <link name='front_left_wheel'>
+    <inertial>
+      <mass value="1.0" />
+      <origin xyz="0 0 0" rpy="0 1.5707 1.5707" />
+      <inertia ixx="0.004133" ixy="0" ixz="0" iyy="0.004133" iyz="0" izz="0.0072" />
+    </inertial>
+    <collision>
+      <origin xyz="0 0 0" rpy="0 1.5707 1.5707" />
+      <geometry>
+        <cylinder radius=".12" length=".08" />
+      </geometry>
+    </collision>
+    <visual name='front_left_wheel_visual'>
+      <origin xyz="0 0 0" rpy="0 1.5707 1.5707" />
+      <geometry>
+        <cylinder radius=".12" length=".08" />
+      </geometry>
+      <material name="black">
+        <color rgba="0.0 0.0 0.0 1.0" />
+      </material>
+    </visual>
+  </link>
+  <joint type="continuous" name="rear_left_wheel_joint">
+    <origin xyz="-0.35 0.3 0" rpy="0 0 0" />
+    <child link="rear_left_wheel" />
+    <parent link="base_link" />
+    <axis xyz="0 1 0" rpy="0 0 0" />
+    <limit effort="100" velocity="10" />
+    <dynamics damping="3.0" friction="3.0" />
+  </joint>
+  <link name='rear_left_wheel'>
+    <inertial>
+      <mass value="1.0" />
+      <origin xyz="0 0 0" rpy="0 1.5707 1.5707" />
+      <inertia ixx="0.004133" ixy="0" ixz="0" iyy="0.004133" iyz="0" izz="0.0072" />
+    </inertial>
+    <collision>
+      <origin xyz="0 0 0" rpy="0 1.5707 1.5707" />
+      <geometry>
+        <cylinder radius=".12" length=".08" />
+      </geometry>
+    </collision>
+    <visual name='rear_left_wheel_visual'>
+      <origin xyz="0 0 0" rpy="0 1.5707 1.5707" />
+      <geometry>
+        <cylinder radius=".12" length=".08" />
+      </geometry>
+      <material name="black">
+        <color rgba="0.0 0.0 0.0 1.0" />
+      </material>
+    </visual>
+  </link>
+  <joint type="continuous" name="front_right_wheel_joint">
+    <origin xyz="0.35 -0.3 0" rpy="0 0 0" />
+    <child link="front_right_wheel" />
+    <parent link="base_link" />
+    <axis xyz="0 1 0" rpy="0 0 0" />
+    <limit effort="100" velocity="10" />
+    <dynamics damping="3.0" friction="3.0" />
+  </joint>
+  <link name='front_right_wheel'>
+    <inertial>
+      <mass value="1.0" />
+      <origin xyz="0 0 0" rpy="0 1.5707 1.5707" />
+      <inertia ixx="0.004133" ixy="0" ixz="0" iyy="0.004133" iyz="0" izz="0.0072" />
+    </inertial>
+    <collision>
+      <origin xyz="0 0 0" rpy="0 1.5707 1.5707" />
+      <geometry>
+        <cylinder radius=".12" length=".08" />
+      </geometry>
+    </collision>
+    <visual name='front_right_wheel_visual'>
+      <origin xyz="0 0 0" rpy="0 1.5707 1.5707" />
+      <geometry>
+        <cylinder radius=".12" length=".08" />
+      </geometry>
+      <material name="black">
+        <color rgba="0.0 0.0 0.0 1.0" />
+      </material>
+    </visual>
+  </link>
+  <joint type="continuous" name="rear_right_wheel_joint">
+    <origin xyz="-0.35 -0.3 0" rpy="0 0 0" />
+    <child link="rear_right_wheel" />
+    <parent link="base_link" />
+    <axis xyz="0 1 0" rpy="0 0 0" />
+    <limit effort="100" velocity="10" />
+    <dynamics damping="3.0" friction="3.0" />
+  </joint>
+  <link name='rear_right_wheel'>
+    <inertial>
+      <mass value="1.0" />
+      <origin xyz="0 0 0" rpy="0 1.5707 1.5707" />
+      <inertia ixx="0.004133" ixy="0" ixz="0" iyy="0.004133" iyz="0" izz="0.0072" />
+    </inertial>
+    <collision>
+      <origin xyz="0 0 0" rpy="0 1.5707 1.5707" />
+      <geometry>
+        <cylinder radius=".12" length=".08" />
+      </geometry>
+    </collision>
+    <visual name='rear_right_wheel_visual'>
+      <origin xyz="0 0 0" rpy="0 1.5707 1.5707" />
+      <geometry>
+        <cylinder radius=".12" length=".08" />
+      </geometry>
+      <material name="black">
+        <color rgba="0.0 0.0 0.0 1.0" />
+      </material>
+    </visual>
+  </link>
+  <joint name="laser_joint" type="fixed">
+    <parent link="base_link" />
+    <child link="laser_frame" />
+    <origin xyz="0.3 0 0.07" rpy="0 0 0" />
+  </joint>
+  <link name="laser_frame">
+    <inertial>
+      <mass value="0.1" />
+      <origin xyz="0 0 0" rpy="0 0 0" />
+      <inertia ixx="0.0001" ixy="0.0" ixz="0.0" iyy="0.0001" iyz="0.0" izz="0.0002" />
     </inertial>
     <visual>
-      <geometry>
-        <box size="0.1 0.3 0.7"/>
-      </geometry>
-    </visual>
-    <collision>
-      <geometry>
-        <box size="0.1 0.3 0.75"/>
-      </geometry>
-    </collision>
-  </link> -->
-  <!-- <joint name="stand_panel_joint" type="fixed">
-    <parent link="base_link"/>
-    <child link="stand_panel"/>
-    <origin xyz="-0.45 0 0.4" rpy="0 0 0" />
-  </joint>   -->
-  <!-- STEP 3 - Wheels -->
-  <joint type="continuous" name="front_left_wheel_joint">
-    <origin xyz="0.35 0.3 0" rpy="0 0 0"/>
-    <child link="front_left_wheel"/>
-    <parent link="base_link"/>
-    <axis xyz="0 1 0" rpy="0 0 0"/>
-    <limit effort="100" velocity="10"/>
-    <dynamics damping="1.0" friction="1.0"/>
-  </joint>
-  <link name='front_left_wheel'>
-    <inertial>
-      <mass value="5.0"/>
-      <origin xyz="0 0 0" rpy="0 1.5707 1.5707"/>
-      <inertia
-          ixx="0.014" ixy="0" ixz="0"
-          iyy="0.014" iyz="0"
-          izz="0.025"
-      />
-    </inertial>
-    <collision>
-      <origin xyz="0 0 0" rpy="0 1.5707 1.5707"/>
-      <geometry>
-        <cylinder radius=".1" length=".08"/>
-      </geometry>
-    </collision>
-    <visual name='front_left_wheel_visual'>
-      <origin xyz="0 0 0" rpy="0 1.5707 1.5707"/>
-      <geometry>
-        <cylinder radius=".1" length=".08"/>
-      </geometry>
-      <material name="black">
-         <color rgba="0.0 0.0 0.0 1.0"/>
-      </material>
-    </visual>
-  </link>
-  <joint type="continuous" name="rear_left_wheel_joint">
-    <origin xyz="-0.35 0.3 0" rpy="0 0 0"/>
-    <child link="rear_left_wheel"/>
-    <parent link="base_link"/>
-    <axis xyz="0 1 0" rpy="0 0 0"/>
-    <limit effort="100" velocity="10"/>
-    <dynamics damping="1.0" friction="1.0"/>
-  </joint>
-  <link name='rear_left_wheel'>
-    <inertial>
-      <mass value="5.0"/>
-      <origin xyz="0 0 0" rpy="0 1.5707 1.5707"/>
-      <inertia
-          ixx="0.014" ixy="0" ixz="0"
-          iyy="0.014" iyz="0"
-          izz="0.025"
-      />
-    </inertial>
-    <collision>
-      <origin xyz="0 0 0" rpy="0 1.5707 1.5707"/>
-      <geometry>
-        <cylinder radius=".1" length=".08"/>
-      </geometry>
-    </collision>
-    <visual name='rear_left_wheel_visual'>
-      <origin xyz="0 0 0" rpy="0 1.5707 1.5707"/>
-      <geometry>
-        <cylinder radius=".1" length=".08"/>
-      </geometry>
-      <material name="black">
-          <color rgba="0.0 0.0 0.0 1.0"/>
-      </material>
-    </visual>
-  </link>
-  <joint type="continuous" name="front_right_wheel_joint">
-    <origin xyz="0.35 -0.3 0" rpy="0 0 0"/>
-    <child link="front_right_wheel"/>
-    <parent link="base_link"/>
-    <axis xyz="0 1 0" rpy="0 0 0"/>
-    <limit effort="100" velocity="10"/>
-    <dynamics damping="1.0" friction="1.0"/>
-  </joint>
-  <link name='front_right_wheel'>
-    <inertial>
-      <mass value="5.0"/>
-      <origin xyz="0 0 0" rpy="0 1.5707 1.5707"/>
-      <inertia
-          ixx="0.014" ixy="0" ixz="0"
-          iyy="0.014" iyz="0"
-          izz="0.025"
-      />
-    </inertial>
-    <collision>
-      <origin xyz="0 0 0" rpy="0 1.5707 1.5707"/>
-      <geometry>
-        <cylinder radius=".1" length=".08"/>
-      </geometry>
-    </collision>
-    <visual name='front_right_wheel_visual'>
-      <origin xyz="0 0 0" rpy="0 1.5707 1.5707"/>
-      <geometry>
-        <cylinder radius=".1" length=".08"/>
-      </geometry>
-      <material name="black">
-          <color rgba="0.0 0.0 0.0 1.0"/>
-      </material>
-    </visual>
-  </link>
-  <joint type="continuous" name="rear_right_wheel_joint">
-    <origin xyz="-0.35 -0.3 0" rpy="0 0 0"/>
-    <child link="rear_right_wheel"/>
-    <parent link="base_link"/>
-    <axis xyz="0 1 0" rpy="0 0 0"/>
-    <limit effort="100" velocity="10"/>
-    <dynamics damping="1.0" friction="1.0"/>
-  </joint>
-  <link name='rear_right_wheel'>
-    <inertial>
-      <mass value="5.0"/>
-      <origin xyz="0 0 0" rpy="0 1.5707 1.5707"/>
-      <inertia
-          ixx="0.014" ixy="0" ixz="0"
-          iyy="0.014" iyz="0"
-          izz="0.025"
-      />
-    </inertial>
-    <collision>
-      <origin xyz="0 0 0" rpy="0 1.5707 1.5707"/>
-      <geometry>
-        <cylinder radius=".1" length=".08"/>
-      </geometry>
-    </collision>
-    <visual name='rear_right_wheel_visual'>
-      <origin xyz="0 0 0" rpy="0 1.5707 1.5707"/>
-      <geometry>
-        <cylinder radius=".1" length=".05"/>
-      </geometry>
-      <material name="black">
-          <color rgba="0.0 0.0 0.0 1.0"/>
-      </material>
-    </visual>
+      <origin xyz="0 0 0" />
+      <geometry>
+        <cylinder length="0.04" radius="0.05" />
+      </geometry>
+      <material name="laser_material">
+        <color rgba="0.13 0.13 0.13 1.0" />
+      </material>
+    </visual>
+    <collision>
+      <origin xyz="0 0 0" />
+      <geometry>
+        <cylinder length="0.04" radius="0.05" />
+      </geometry>
+    </collision>
   </link>
   <!-- STEP 6 - Gazebo frictions and colors -->
-  <gazebo reference="front_left_wheel">
-    <mu1>1.5</mu1>
-    <mu2>0.7</mu2>
-    <kp>200000.0</kp>
-    <kd>5000.0</kd>
-    <minDepth>0.002</minDepth>
-    <maxVel>0.3</maxVel>
-    <fdir1>0 1 0</fdir1>
-    <!-- <material>Gazebo/Green</material> -->
-  </gazebo>
-  <gazebo reference="front_right_wheel">
-    <mu1>1.5</mu1>
-    <mu2>0.7</mu2>
-    <kp>200000.0</kp>
-    <kd>5000.0</kd>
-    <minDepth>0.002</minDepth>
-    <maxVel>0.3</maxVel>
-    <fdir1>0 1 0</fdir1>
-    <!-- <material>Gazebo/Green</material> -->
-  </gazebo>
-  <gazebo reference="rear_left_wheel">
-    <mu1>1.5</mu1>
-    <mu2>0.7</mu2>
-    <kp>200000.0</kp>
-    <kd>5000.0</kd>
-    <minDepth>0.002</minDepth>
-    <maxVel>0.3</maxVel>
-    <fdir1>0 1 0</fdir1>
-    <!-- <material>Gazebo/Green</material> -->
-  </gazebo>
-  <gazebo reference="rear_right_wheel">
-    <mu1>1.5</mu1>
-    <mu2>0.7</mu2>
-    <kp>200000.0</kp>
-    <kd>5000.0</kd>
-    <minDepth>0.002</minDepth>
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