Commit message: cart_description package not needed anymore + tf frames and hardware package modified

File: cart_navigation/urdf/lidar.xacro (robot description, xacro)
@@ -4,5 +4,5 @@
      <parent link="base_link"/>
      <child link="laser_frame"/>
-     <origin xyz="0.3 0 0.075" rpy="0 0 0"/>
+     <origin xyz="0.12 0 0.075" rpy="0 0 0"/>
    </joint>
    <link name="laser_frame">

File: hardware_navigation/urdf/cart.urdf.xacro (robot description, xacro)
@@ -1,6 +1,6 @@
 <?xml version="1.0"?>
 <robot name="cart" xmlns:xacro="http://www.ros.org/wiki/xacro">
-    <xacro:include filename="cart_design.xacro" />
+    <xacro:include filename="cart_design.urdf.xacro" />
     <xacro:include filename="cart_control.gazebo"/>
-    <!-- <xacro:include filename="lidar.xacro" /> -->
+    <xacro:include filename="lidar.xacro"/>
 </robot>
