Commit message: new 4 wheel and other modifications

File: cart_navigation/urdf/cart.urdf.xacro (robot description, xacro)
@@ -1,6 +1,8 @@
 <?xml version="1.0"?>
 <robot name="cart" xmlns:xacro="http://www.ros.org/wiki/xacro">
-    <xacro:include filename="cart_design.xacro" />
-    <xacro:include filename="cart_control.gazebo"/>
+    <!-- <xacro:include filename="cart_design.xacro" /> -->
+    <!-- <xacro:include filename="cart_control.gazebo"/> -->
+    <xacro:include filename="4_wheel.urdf.xacro" />
+    <xacro:include filename="control.gazebo"/>
     <!-- <xacro:include filename="lidar.xacro" /> -->
 </robot>

File: hardware_navigation/urdf/cart_design.urdf.xacro (robot description, xacro)
@@ -6,12 +6,12 @@
   <!-- Robot Constants -->
   <xacro:property name="base_width" value="0.2"/>
-  <xacro:property name="base_length" value="0.4"/>
-  <xacro:property name="base_height" value="0.1"/>
-  <xacro:property name="wheel_radius" value="0.06"/>
+  <xacro:property name="base_length" value="0.3"/>
+  <xacro:property name="base_height" value="0.03"/>
+  <xacro:property name="wheel_radius" value="0.0325"/>
   <xacro:property name="wheel_width" value="0.03"/>
-  <xacro:property name="wheel_ygap" value="0.02"/>
-  <xacro:property name="wheel_zoff" value="0.03"/>
-  <xacro:property name="wheel_xoff" value="0.12"/>
-  <xacro:property name="caster_xoff" value="0.14"/>
+  <xacro:property name="wheel_ygap" value="0.015"/>
+  <xacro:property name="wheel_zoff" value="0.015"/>
+  <xacro:property name="wheel_xoff" value="0.1"/>
+  <xacro:property name="caster_xoff" value="0.1"/>
   <!-- Robot Footprint -->
   <link name="base_footprint"/>

File: hardware_navigation/urdf/lidar.xacro (robot description, xacro)
@@ -5,5 +5,5 @@
     <parent link="base_link"/>
     <child link="laser_frame"/>
-    <origin xyz="0.12 0 0.075" rpy="0 0 0"/>
+    <origin xyz="0.1 0 0.025" rpy="0 0 0"/>
   </joint>
   <link name="laser_frame">
