Commit message: Initial fresh repo

File: cart_navigation/urdf/2w_cart.urdf.xacro (robot description, xacro)
@@ -10,8 +10,8 @@
   <xacro:property name="base_length" value="0.3"/>
   <xacro:property name="base_height" value="0.05"/>
-  <xacro:property name="base_mass" value="3"/>
+  <xacro:property name="base_mass" value="2"/>
   <xacro:property name="wheel_radius" value="0.0325"/> <!-- impprtant -->
   <xacro:property name="wheel_width" value="0.03"/>
-  <xacro:property name="wheel_mass" value="0.2"/>
+  <xacro:property name="wheel_mass" value="0.4"/>
   <xacro:property name="wheel_zoff" value="0.0325"/>
   <xacro:property name="wheel_xoff" value="0.1"/>   <!-- impprtant -->

File: cart_navigation/urdf/cart.urdf.xacro (robot description, xacro)
@@ -1,8 +1,5 @@
 <?xml version="1.0"?>
 <robot name="cart" xmlns:xacro="http://www.ros.org/wiki/xacro">
-    <!-- <xacro:include filename="cart_design.xacro" /> -->
-    <!-- <xacro:include filename="cart_control.gazebo"/> -->
-    <xacro:include filename="4_wheel.urdf.xacro" />
-    <xacro:include filename="control.gazebo"/>
-    <!-- <xacro:include filename="lidar.xacro" /> -->
+    <!-- <xacro:include filename="$(find cart_navigation)/urdf/4w_cart.urdf.xacro"/> -->
+    <xacro:include filename="$(find cart_navigation)/urdf/2w_cart.urdf.xacro"/>
 </robot>

File: cart_navigation/urdf/lidar.xacro (robot description, xacro)
@@ -1,52 +1,78 @@
 <?xml version="1.0"?>
-<robot xmlns:xacro="http://www.ros.org/wiki/xacro" >
-   <joint name="laser_joint" type="fixed">
-     <parent link="base_link"/>
-     <child link="laser_frame"/>
-     <origin xyz="0.12 0 0.075" rpy="0 0 0"/>
-   </joint>
-   <link name="laser_frame">
+<robot xmlns:xacro="http://www.ros.org/wiki/xacro">
+  <xacro:macro name="lidar_sensor" params="
+    prefix:=''
+    parent:='base_link'
+    frame_id:='laser_frame'
+    xyz_offset
+    rpy_offset
+    lidar_width:=0.03
+    lidar_height:=0.03
+    mass:=0.085
+    color:='red'
+    update_rate:=10
+    ray_count:=360
+    min_angle:='-3.14159'
+    max_angle:='3.14159'
+    min_range:='0.20'
+    max_range:='30.0'
+    range_resolution:='0.013'
+    topic_name:='scan'
+    always_on:=true
+    visualize:=false
+    enable_collision:=false">
+    <link name="${prefix}${frame_id}">
       <visual>
-         <origin xyz="0 0 0"/>
-         <geometry>
-            <cylinder length="0.04" radius="0.05"/>
-         </geometry>
-         <material name="laser_material">
-            <color rgba="0.13 0.13 0.13 1.0"/>
-         </material>
+        <origin xyz="0 0 0" rpy="0 0 0"/>
+        <geometry>
+          <cylinder radius="${lidar_width / 2}" length="${lidar_height}"/>
+        </geometry>
+        <material name="${color}"/>
       </visual>
-      <collision>
-         <origin xyz="0 0 0"/>
-         <geometry>
-            <cylinder length="0.04" radius="0.05"/>
-         </geometry>
-      </collision>
-      <xacro:inertial_cylinder mass="0.1" length="0.04" radius="0.05">
-         <origin xyz="0 0 0" rpy="0 0 0"/>
-      </xacro:inertial_cylinder>
-   </link>
-   <!-- 2D Lidar New Gazebo Sensor Plugin  -->
-   <gazebo reference="laser_frame">
-      <sensor name="laser" type="gpu_lidar">
-         <pose> 0 0 0 0 0 0 </pose>
-         <always_on>true</always_on>
-         <visualize>true</visualize>
-         <update_rate>10</update_rate>
-         <topic>scan</topic>
-         <gz_frame_id>laser_frame</gz_frame_id>
-         <lidar>
-            <scan>
-               <horizontal>
-               <samples>360</samples>
-               <min_angle>-3.14</min_angle>
-               <max_angle>3.14</max_angle>
-               </horizontal>
-            </scan>
-            <range>
-               <min>0.3</min>
-               <max>12</max>
-            </range>
-         </lidar>
+      <xacro:if value="${enable_collision}">
+        <collision>
+          <origin xyz="0 0 0" rpy="0 0 0"/>
+          <geometry>
+            <cylinder radius="${lidar_width / 2}" length="${lidar_height}"/>
+          </geometry>
+        </collision>
+      </xacro:if>
+      <xacro:cylinder_inertia m="${mass}" r="${lidar_width / 2}" h="${lidar_height}"/>
+    </link>
+    <joint name="${prefix}${frame_id}_joint" type="fixed">
+      <parent link="${prefix}${parent}"/>
+      <child link="${prefix}${frame_id}"/>
+      <origin xyz="${xyz_offset}" rpy="${rpy_offset}"/>
+    </joint>
+    <gazebo reference="${prefix}${frame_id}">
+      <sensor name="${prefix}lidar_sensor" type="gpu_lidar">
+        <topic>${topic_name}</topic>
+        <update_rate>${update_rate}</update_rate>
+        <always_on>${always_on}</always_on>
+        <visualize>${visualize}</visualize>
+        <ray>
+          <scan>
+            <horizontal>
+              <samples>${ray_count}</samples>
+              <resolution>1</resolution>
+              <min_angle>${min_angle}</min_angle>
+              <max_angle>${max_angle}</max_angle>
+            </horizontal>
+            <vertical>
+              <samples>1</samples>
+              <resolution>1</resolution>
+              <min_angle>0</min_angle>
+              <max_angle>0</max_angle>
+            </vertical>
+          </scan>
+          <range>
+            <min>${min_range}</min>
+            <max>${max_range}</max>
+            <resolution>${range_resolution}</resolution>
+          </range>
+        </ray>
+        <gz_frame_id>${prefix}${frame_id}</gz_frame_id>
       </sensor>
-   </gazebo>
+    </gazebo>
+  </xacro:macro>
 </robot>

File: cart_navigation/urdf/macros.xacro (robot description, xacro)
@@ -17,3 +17,11 @@
     </inertial>
   </xacro:macro>
+  <xacro:macro name="sphere_inertia" params="m r">
+  <inertial>
+    <mass value="${m}"/>
+    <inertia ixx="${(2/5) * m * (r*r)}" ixy="0.0" ixz="0.0"
+             iyy="${(2/5) * m * (r*r)}" iyz="0.0"
+             izz="${(2/5) * m * (r*r)}"/>
+  </inertial>
+  </xacro:macro>
 </robot>

File: hardware_navigation/urdf/cart.urdf.xacro (robot description, xacro)
@@ -1,6 +1,4 @@
 <?xml version="1.0"?>
 <robot name="cart" xmlns:xacro="http://www.ros.org/wiki/xacro">
-    <xacro:include filename="cart_design.urdf.xacro" />
-    <xacro:include filename="cart_control.gazebo"/>
-    <xacro:include filename="lidar.xacro"/>
+    <xacro:include filename="$(find hardware_navigation)/urdf/cart_design.urdf.xacro"/>
 </robot>

File: hardware_navigation/urdf/lidar.xacro (robot description, xacro)
@@ -1,54 +1,78 @@
 <?xml version="1.0"?>
-<robot xmlns:xacro="http://www.ros.org/wiki/xacro" >
-  <!-- Laser LIDAR Sensor -->
-  <joint name="laser_joint" type="fixed">
-    <parent link="base_link"/>
-    <child link="laser_frame"/>
-    <origin xyz="0.1 0 0.025" rpy="0 0 0"/>
-  </joint>
-  <link name="laser_frame">
-    <visual>
-      <origin xyz="0 0 0"/>
-      <geometry>
-        <cylinder length="0.02" radius="0.02"/>
-      </geometry>
-      <material name="red">
-        <color rgba="0.8 0.0 0.0 1.0"/>
-      </material>
-    </visual>
-    <collision>
-      <origin xyz="0 0 0"/>
-      <geometry>
-        <cylinder length="0.02" radius="0.02"/>
-      </geometry>
-    </collision>
-    <inertial>
-      <mass value="0.1"/>
-      <origin xyz="0 0 0" rpy="0 0 0"/>
-      <inertia ixx="0.0001" ixy="0.0" ixz="0.0" iyy="0.0001" iyz="0.0" izz="0.0002"/>
-    </inertial>
-  </link>
-  <gazebo reference="laser_frame">
-    <sensor name="laser" type="gpu_lidar">
-      <pose>0 0 0 0 0 0</pose>
-      <always_on>true</always_on>
-      <visualize>true</visualize>
-      <update_rate>10</update_rate>
-      <topic>scan</topic>
-      <gz_frame_id>laser_frame</gz_frame_id>
-      <lidar>
-        <scan>
-          <horizontal>
-            <samples>360</samples>
-            <min_angle>-3.14</min_angle>
-            <max_angle>3.14</max_angle>
-          </horizontal>
-        </scan>
-        <range>
-          <min>0.3</min>
-          <max>12</max>
-        </range>
-      </lidar>
-    </sensor>
-  </gazebo>
+<robot xmlns:xacro="http://www.ros.org/wiki/xacro">
+  <xacro:macro name="lidar_sensor" params="
+    prefix:=''
+    parent:='base_link'
+    frame_id:='laser_frame'
+    xyz_offset
+    rpy_offset
+    lidar_width:=0.03
+    lidar_height:=0.03
+    mass:=0.085
+    color:='red'
+    update_rate:=10
+    ray_count:=360
+    min_angle:='-3.14159'
+    max_angle:='3.14159'
+    min_range:='0.20'
+    max_range:='30.0'
+    range_resolution:='0.013'
+    topic_name:='scan'
+    always_on:=true
+    visualize:=false
+    enable_collision:=false">
+    <link name="${prefix}${frame_id}">
+      <visual>
+        <origin xyz="0 0 0" rpy="0 0 0"/>
+        <geometry>
+          <cylinder radius="${lidar_width / 2}" length="${lidar_height}"/>
+        </geometry>
+        <material name="${color}"/>
+      </visual>
+      <xacro:if value="${enable_collision}">
+        <collision>
+          <origin xyz="0 0 0" rpy="0 0 0"/>
+          <geometry>
+            <cylinder radius="${lidar_width / 2}" length="${lidar_height}"/>
+          </geometry>
+        </collision>
+      </xacro:if>
+      <xacro:cylinder_inertia m="${mass}" r="${lidar_width / 2}" h="${lidar_height}"/>
+    </link>
+    <joint name="${prefix}${frame_id}_joint" type="fixed">
+      <parent link="${prefix}${parent}"/>
+      <child link="${prefix}${frame_id}"/>
+      <origin xyz="${xyz_offset}" rpy="${rpy_offset}"/>
+    </joint>
+    <gazebo reference="${prefix}${frame_id}">
+      <sensor name="${prefix}lidar_sensor" type="gpu_lidar">
+        <topic>${topic_name}</topic>
+        <update_rate>${update_rate}</update_rate>
+        <always_on>${always_on}</always_on>
+        <visualize>${visualize}</visualize>
+        <ray>
+          <scan>
+            <horizontal>
+              <samples>${ray_count}</samples>
+              <resolution>1</resolution>
+              <min_angle>${min_angle}</min_angle>
+              <max_angle>${max_angle}</max_angle>
+            </horizontal>
+            <vertical>
+              <samples>1</samples>
+              <resolution>1</resolution>
+              <min_angle>0</min_angle>
+              <max_angle>0</max_angle>
+            </vertical>
+          </scan>
+          <range>
+            <min>${min_range}</min>
+            <max>${max_range}</max>
+            <resolution>${range_resolution}</resolution>
+          </range>
+        </ray>
+        <gz_frame_id>${prefix}${frame_id}</gz_frame_id>
+      </sensor>
+    </gazebo>
+  </xacro:macro>
 </robot>

File: hardware_navigation/urdf/macros.xacro (robot description, xacro)
@@ -18,8 +18,10 @@
   </xacro:macro>
   <xacro:macro name="sphere_inertia" params="m r">
-    <inertial>
-      <mass value="${m}"/>
-      <inertia ixx="${(2/5) * m * (r*r)}" ixy="0.0" ixz="0.0" iyy="${(2/5) * m * (r*r)}" iyz="0.0" izz="${(2/5) * m * (r*r)}"/>
-    </inertial>
+  <inertial>
+    <mass value="${m}"/>
+    <inertia ixx="${(2/5) * m * (r*r)}" ixy="0.0" ixz="0.0"
+             iyy="${(2/5) * m * (r*r)}" iyz="0.0"
+             izz="${(2/5) * m * (r*r)}"/>
+  </inertial>
   </xacro:macro>
 </robot>

Commit message: bt behavior files added for + robot position adjusted

File: cart_navigation/urdf/2w_cart.urdf.xacro (robot description, xacro)
@@ -26,5 +26,5 @@
     <parent link="base_footprint"/>
     <child link="base_link"/>
-    <origin xyz="0.0 0.0 ${-(wheel_radius + 0.06) + 0.005}" rpy="0 0 0"/>
+    <origin xyz="0.0 0.0 ${2 * wheel_radius}" rpy="0 0 0"/>
   </joint>
   <!-- Base -->
